File: Board/v2/v2.brd (EAGLE design)
At the start: 88.5 x 48.5 mm, 63 parts, among them IC2 PCF8574TS, Q1 BSA223SP, Q2 BSA223SP, SW1 EVQQ, SW2 EVQQ, SW3 EVQQ, SW4 EVQQ, U2 BME680

Commit message: Updating Board
New version of board with several changes and new CCS811 sensor
Parts:
- removed JMP1: 0R-JUMPC, jump-0r-smd:C0R-JMP
- removed JP2: (no value), microbuilder:1X05_ROUND_70
- removed LED1, LED2, LED3, LED4: (no value), led:CHIPLED_0805
- removed Q2: BSA223SP, transistor-fet:SC75_INFINEON
- removed R10, R18: 10k, rcl:R0805
- removed SJ1, SJ2: (no value), microbuilder:SOLDERJUMPER_CLOSEDWIRE
- removed SW4: EVQQ, microbuilder:EVQ-Q2_SMALLER
- added C5: 100n, rcl:C0805
- added R20: 10k, rcl:R0805
- added RESET: EVQQ, adafruit:EVQ-Q2
- added SWCLK, SWDIO: (no value), wirepad:SMD1,27-2,54
- added U$33: MAX17043, MAX17043:DFN-2X3
- added U$5: LED_LIGHTGUIDE, 000_Simons_Eigene:LPA-C041301S-X
- added X1: 20317, microbuilder:2X05_1.27MM_BOX_POSTS
- Q1: value BSA223SP -> DMG3415; device transistor-fet:SC75_INFINEON -> microbuilder:SOT23-WIDE
- SW1, SW2, SW3: device microbuilder:EVQ-Q2_SMALLER -> adafruit:EVQ-Q2
- U$8: value (none) -> MSK-12C02_SMD_SPDT_SWITCH; device MSK-12C02 SMD Micro Slider Switch SPDT:MSK-12C02 -> 000_Simons_Eigene:MSK-12C02
- moved C1 18.5 mm to (-6.90, 35.1), flipped to the top, turned to 270 degrees
- moved U2 14.8 mm to (-5.62, 35.1), turned to 270 degrees
- moved Q1 14.5 mm to (73.6, 35.1), flipped to the top, turned to 270 degrees
- moved SW3 8.47 mm to (78.0, -6.50)
- moved R9 8.35 mm to (77.8, -5.50)
- moved R6 7.53 mm to (26.7, -8.38), flipped to the bottom, turned to 180 degrees
- moved SW2 5.97 mm to (66.5, -6.50)
- moved R8 5.85 mm to (66.3, -5.50)
- moved R5 4.57 mm to (21.6, -8.38), flipped to the bottom, turned to 180 degrees
- moved R19 4.02 mm to (66.4, 19.9), turned to 180 degrees
- moved SW1 3.50 mm to (55.0, -6.50)
- moved R3 3.42 mm to (70.6, 35.1)
- moved U$8 3.35 mm to (88.1, 13.0)
- moved R7 3.35 mm to (54.8, -5.50)
- moved R14 2.97 mm to (3.48, 29.0), turned to 0 degrees
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Connections:
- net N$7 renamed EN
- removed net DELAY: IC2.14, JP2.3, PAD12.1, PAD6.1, Q1.2, R10.2, SW4.A, SW4.A'
- removed net DONE: JP2.5, U$15.13
- removed net ENOUT: JP2.4, SJ1.2, U$8.L2
- removed net N$20: IC2.20, R1.2
- removed net N$21: IC2.19, R2.2
- removed net N$22: IC2.17, R5.2
- removed net N$23: IC2.16, R6.2
- removed net N$24: LED4.A, R6.1
- removed net N$25: LED3.A, R5.1
- removed net N$26: LED2.A, R2.1
- removed net N$27: LED1.A, R1.1
- new net BAT_ALERT: R20.1, U$15.A4, U$33.5
- new net LI_BAT: U$15.BAT, U$33.2
- new net MANUAL_INT: IC2.12, PAD12.1, PAD6.1, R9.2, SW3.A, SW3.A', U$15.A3
- new net N$10: IC2.19, R5.1
- new net N$11: IC2.20, R6.1
- new net N$14: SWDIO.1, X1.2
- new net N$15: SWCLK.1, X1.4
- new net N$16: R5.2, U$5.C3
- new net N$17: R2.2, U$5.C2
- new net N$18: R1.2, U$5.C1
- net 3.3V: now also C5.1, Q1.2, R20.2, U$33.3, U$5.A1, U$5.A2, U$5.A3, U$5.A4, U$8.L2, X1.1; no longer JMP1.1, Q1.3, Q2.3, SJ1.1, SW4.B, SW4.B'
- net BUZZER: now also Q1.1; no longer Q2.1
- net GND: now also C5.2, RESET.B, RESET.B', U$33.1, U$33.4, U$33.6, U$33.EXP, X1.3, X1.5, X1.9; no longer JP2.2, LED1.C, LED2.C, LED3.C, LED4.C, R10.1, R18.2
- net N$1: now also IC2.16, R1.1; no longer JMP1.2, JP2.1
- net N$12: no longer R18.1
- net N$13: now also R6.2, U$5.C4; no longer IC2.12, R9.2, SW3.A, SW3.A'
- net N$2: now also IC2.17, R2.1; no longer Q1.1, R19.1, SJ2.1
- net N$8: now also Q1.3; no longer Q2.2
- net RST: now also RESET.A, RESET.A', X1.10
- net RTC_INT: now also R19.1; no longer SJ2.2
- net SCL: now also U$33.7
- net SDA: now also U$33.8
- net VBAT: no longer JMP1.3
Routing:
- net DELAY: track 145.3 -> 0.00 mm, vias 4 -> 0
- net MANUAL_INT: track 0.00 -> 121.5 mm, vias 0 -> 5
- net 3.3V: track 296.6 -> 357.6 mm, vias 11 -> 13
- net VBAT: track 75.8 -> 23.5 mm
- net RST: track 73.3 -> 111.8 mm, vias 1 -> 4
- net N$13: track 38.6 -> 3.44 mm, vias 2 -> 1
- net BAT_ALERT: track 0.00 -> 33.7 mm, vias 0 -> 1
- net N$1: track 4.42 -> 33.3 mm
- net N$20: track 26.0 -> 0.00 mm, vias 1 -> 0
- net ENOUT: track 24.9 -> 0.00 mm
- net N$2: track 3.85 -> 25.7 mm
- net LI_BAT: track 0.00 -> 20.2 mm, vias 0 -> 1
- net N$21: track 18.8 -> 0.00 mm, vias 1 -> 0
- net N$10: track 0.00 -> 17.4 mm
- net SDA: track 110.5 -> 125.6 mm, vias 5 -> 6
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Other:
- board size 88.5 x 48.5 mm -> 98 x 48.5 mm
- board text added: "BME680 datalogger v2 06.01.2018 Simon Gaßner"
- board text added: "I2C_INT"
- board text added: "MAN_INT"
- board text added: "RX"
- board text added: "TX"
- board text removed: "BAT/3.3V"
- board text removed: "BME680 datalogger v1 24.11.2017 Simon Gaßner"
- board text removed: "Delay"
- board text removed: "Done"
- board text removed: "ENout"
- board text removed: "VDD"
