File: Board/v3/v3.brd (EAGLE design)
At the start: 88.5 x 48.5 mm, 63 parts, among them IC2 PCF8574TS, Q1 BSA223SP, Q2 BSA223SP, SW1 EVQQ, SW2 EVQQ, SW3 EVQQ, SW4 EVQQ, U2 BME680

Commit message: Updating Board
New version of board with several changes and new CCS811 sensor
Parts:
- removed JMP1: 0R-JUMPC, jump-0r-smd:C0R-JMP
- removed JP2: (no value), microbuilder:1X05_ROUND_70
- removed JP5: (no value), pinhead-2:1X04
- removed LED1, LED2, LED3, LED4: (no value), led:CHIPLED_0805
- removed Q2: BSA223SP, transistor-fet:SC75_INFINEON
- removed SJ1, SJ2: (no value), microbuilder:SOLDERJUMPER_CLOSEDWIRE
- removed SW4: EVQQ, microbuilder:EVQ-Q2_SMALLER
- added C5: 100n, rcl:C0805
- added C6: 4u7, rcl:C0805
- added C7: 1u, rcl:C0805
- added R20: 10k, rcl:R0805
- added R21, R22, R23, R24: 100k, rcl:R0805
- added RESET: EVQQ, adafruit:EVQ-Q2
- added SWCLK, SWDIO: (no value), wirepad:SMD1,27-2,54
- added U$33: MAX17043, MAX17043:DFN-2X3
- added U$5: LED_LIGHTGUIDE, 000_Simons_Eigene:LPA-C041301S-X
- added U1: CCS811, CCS811_Breakout_Temp:LGA10
- added X1: 20317, microbuilder:2X05_1.27MM_BOX_POSTS
- JP6: device pinhead-2:1X04 -> pinhead-2:1X04/90
- Q1: value BSA223SP -> DMG3415; device transistor-fet:SC75_INFINEON -> microbuilder:SOT23-WIDE
- R10: value 10k -> 1k
- R18: value 10k -> 19k
- R4: value 10k -> 10R
- SW1, SW2, SW3: device microbuilder:EVQ-Q2_SMALLER -> adafruit:EVQ-Q2
- U$8: value (none) -> MSK-12C02_SMD_SPDT_SWITCH; device MSK-12C02 SMD Micro Slider Switch SPDT:MSK-12C02 -> 000_Simons_Eigene:MSK-12C02
- moved R18 61.7 mm to (62.8, 20.0), turned to 270 degrees
- moved R10 21.8 mm to (71.9, 15.1), turned to 180 degrees
- moved C1 18.5 mm to (-6.90, 35.1), flipped to the top, turned to 270 degrees
- moved U2 14.8 mm to (-5.62, 35.1), turned to 270 degrees
- moved Q1 14.5 mm to (73.6, 35.1), flipped to the top, turned to 270 degrees
- moved R9 9.47 mm to (78.8, -7.48)
- moved SW3 8.47 mm to (78.0, -6.50)
- moved R6 7.63 mm to (26.7, -8.84), flipped to the bottom, turned to 180 degrees
- moved R8 7.05 mm to (67.3, -7.48)
- moved SW2 5.97 mm to (66.5, -6.50)
- moved JP6 5.47 mm to (16.7, 32.0)
- moved R5 4.73 mm to (21.6, -8.84), flipped to the bottom, turned to 180 degrees
- moved R7 4.43 mm to (55.8, -6.72)
- moved R19 4.02 mm to (66.4, 19.9), turned to 180 degrees
- moved SW1 3.50 mm to (55.0, -6.50)
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Connections:
- net N$5 renamed BME_CSB
- net N$6 renamed RTC_INT_
- net N$7 renamed EN
- removed net DELAY: IC2.14, JP2.3, PAD12.1, PAD6.1, Q1.2, R10.2, SW4.A, SW4.A'
- removed net DONE: JP2.5, U$15.13
- removed net ENOUT: JP2.4, SJ1.2, U$8.L2
- removed net N$1: JMP1.2, JP2.1
- removed net N$12: R15.1, R18.1, U2.5
- removed net N$13: IC2.12, R9.2, SW3.A, SW3.A'
- removed net N$2: Q1.1, R19.1, SJ2.1
- removed net N$20: IC2.20, R1.2
- removed net N$21: IC2.19, R2.2
- removed net N$22: IC2.17, R5.2
- removed net N$23: IC2.16, R6.2
- removed net N$24: LED4.A, R6.1
- removed net N$25: LED3.A, R5.1
- removed net N$26: LED2.A, R2.1
- removed net N$27: LED1.A, R1.1
- removed net N$3: IC2.10, R7.2, SW1.A, SW1.A'
- removed net N$4: IC2.11, R8.2, SW2.A, SW2.A'
- new net BAT_ALERT: R20.1, U$15.A4, U$33.5
- new net BME_SDO: R15.1, U2.5
- new net CCS_WAKE: U$15.A0, U1.7
- new net LED1: IC2.16, R1.1, R21.1
- new net LED1_: R1.2, U$5.C1
- new net LED2: IC2.17, R2.1, R22.1
- new net LED2_: R2.2, U$5.C2
- new net LED3: IC2.19, R23.1, R5.1
- new net LED3_: R5.2, U$5.C3
- new net LED4: IC2.20, R24.1, R6.1
- new net LED4_: R6.2, U$5.C4
- new net LI_BAT: R10.2, U$15.BAT
- new net LI_BAT_: C7.1, R10.1, U$33.2
- new net SENSE_PWM: U1.4, U1.5
- new net SW1: IC2.10, R7.1, SW1.B, SW1.B'
- new net SW2: IC2.11, R8.1, SW2.B, SW2.B'
- new net SW3_MANUAL_INT: IC2.12, PAD12.1, PAD6.1, R9.1, SW3.B, SW3.B', U$15.A3
- new net SWCLK: SWCLK.1, X1.4
- new net SWDIO: SWDIO.1, X1.2
- net 3.3V: now also C5.1, C6.1, JP6.1, Q1.2, R18.2, R20.2, R21.2, R22.2, R23.2, R24.2, R7.2, R8.2, R9.2, U$33.3, U$5.A1, U$5.A2, U$5.A3, U$5.A4, U1.6, X1.1; no longer JMP1.1, JP5.4, JP6.4, Q1.3, Q2.3, SJ1.1, SW1.B, SW1.B', SW2.B, SW2.B', SW3.B, SW3.B', SW4.B, SW4.B'
- net BUZZER: now also Q1.1; no longer Q2.1
- net CARD_DET: now also R18.1
- net GND: now also C5.2, C6.2, C7.2, JP6.4, RESET.B, RESET.B', SW1.A, SW1.A', SW2.A, SW2.A', SW3.A, SW3.A', U$33.1, U$33.4, U$33.6, U$33.EXP, U1.EP, X1.3, X1.5, X1.9; no longer JP2.2, JP5.1, JP6.1, LED1.C, LED2.C, LED3.C, LED4.C, R10.1, R18.2, R7.1, R8.1, R9.1
- net N$8: now also Q1.3; no longer Q2.2
- net RST: now also RESET.A, RESET.A', X1.10
- net RTC_INT: now also R19.1; no longer SJ2.2
- net SCL: now also U$33.7, U1.10; no longer JP5.3
- net SDA: now also U$33.8, U1.9; no longer JP5.2
- net VBAT: no longer JMP1.3
Routing:
- net DELAY: track 145.3 -> 0.00 mm, vias 4 -> 0
- net SW3_MANUAL_INT: track 0.00 -> 120.6 mm, vias 0 -> 5
- net CCS_WAKE: track 0.00 -> 100.0 mm, vias 0 -> 2
- net 3.3V: track 296.6 -> 348.8 mm, vias 11 -> 20
- net VBAT: track 75.8 -> 25.9 mm
- net N$13: track 38.6 -> 0.00 mm, vias 2 -> 0
- net SW2: track 0.00 -> 35.1 mm, vias 0 -> 1
- net BAT_ALERT: track 0.00 -> 33.7 mm, vias 0 -> 1
- net LED1: track 0.00 -> 33.1 mm
- net N$4: track 29.1 -> 0.00 mm, vias 2 -> 0
- net RST: track 73.3 -> 101.8 mm, vias 1 -> 4
- net LED2: track 0.00 -> 26.7 mm
- net N$20: track 26.0 -> 0.00 mm, vias 1 -> 0
- net ENOUT: track 24.9 -> 0.00 mm
- net LI_BAT_: track 0.00 -> 23.8 mm, vias 0 -> 1
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Other:
- board size 88.5 x 48.5 mm -> 98 x 48.5 mm
- board text added: "BME680 datalogger v3 26.01.2018 Simon Gaßner"
- board text added: "I2C_INT"
- board text added: "MAN_INT"
- board text added: "RX"
- board text added: "TX"
- board text removed: "BAT/3.3V"
- board text removed: "BME680 datalogger v1 24.11.2017 Simon Gaßner"
- board text removed: "Delay"
- board text removed: "Done"
- board text removed: "ENout"
- board text removed: "VDD"
